File: FVCU.kicad_pcb (KiCad board)
At the start: 2 copper layers, 68 x 60 mm, 14 parts, among them J1 ESP32 Connector, J2 Conn_01x19, J3 MCP2551, J4 Conn_01x14

Commit message: Updated
Parts:
- added C1: C, Capacitor_SMD:C_0805_2012Metric_Pad1.18x1.45mm_HandSolder, F.Cu at (75.8, 86.1)
- added R5: 3K, Resistor_SMD:R_0805_2012Metric, F.Cu at (59.5, 89.9)
- added TP1: TestPoint, TestPoint:TestPoint_Pad_D2.0mm, F.Cu at (49.8, 84.2)
- added TP2: TestPoint, TestPoint:TestPoint_Pad_D2.0mm, F.Cu at (49.8, 89.6)
- added TP3: TestPoint, TestPoint:TestPoint_Pad_D2.0mm, F.Cu at (40.9, 92.6)
- added TP4: TestPoint, TestPoint:TestPoint_Pad_D2.0mm, F.Cu at (40.7, 101.9)
- added TP5: TestPoint, TestPoint:TestPoint_Pad_D2.0mm, F.Cu at (40.7, 109.1)
- moved J1 50.9 mm to (90.7, 93.0), turned to -90 degrees
- moved R4 47.3 mm to (53.8, 111.1), turned to 180 degrees
- moved R3 44.7 mm to (53.8, 105.6), turned to 180 degrees
- moved R2 42.1 mm to (57.9, 111.1), turned to 180 degrees
- moved R1 39.3 mm to (57.8, 105.6), turned to 180 degrees
- moved J3 37.0 mm to (65.5, 88.9), turned to 90 degrees
- moved J2 26.8 mm to (90.7, 116.8)
- moved G*** 1.98 mm to (58.0, 99.8)
Connections:
- J1 pad 19: unconnected-(J1-Pin_19-Pad19) -> GND
- J3 pad 8: GND -> Net-(J3-Pin_8)
- J4 pad 1: +5V -> Net-(J2-Pin_17)
- J4 pad 10: Net-(J2-Pin_15) -> Net-(J4-Pin_10)
- J4 pad 11: Net-(J2-Pin_14) -> CANH
- J4 pad 12: Net-(J2-Pin_13) -> CANL
- J4 pad 13: Net-(J4-Pin_13) -> unconnected-(J4-Pin_13-Pad13)
- J4 pad 14: Net-(J4-Pin_14) -> GND
- J4 pad 2: GND -> Net-(J2-Pin_16)
- J4 pad 3: CANH -> Net-(J2-Pin_15)
- J4 pad 4: CANL -> Net-(J2-Pin_14)
- J4 pad 5: unconnected-(J4-Pin_5-Pad5) -> Net-(J2-Pin_13)
- J4 pad 6: Net-(J2-Pin_17) -> Net-(J4-Pin_6)
- J4 pad 7: Net-(J2-Pin_16) -> unconnected-(J4-Pin_7-Pad7)
- J4 pad 9: unconnected-(J4-Pin_9-Pad9) -> +5V
- R1 pad 2: Net-(J2-Pin_12) -> Net-(J2-Pin_11)
- R2 pad 2: Net-(J2-Pin_11) -> Net-(J2-Pin_12)
- R3 pad 1: Net-(J2-Pin_12) -> Net-(J2-Pin_11)
- R3 pad 2: Net-(J4-Pin_14) -> Net-(J4-Pin_10)
- R4 pad 1: Net-(J2-Pin_11) -> Net-(J2-Pin_12)
- R4 pad 2: Net-(J4-Pin_13) -> Net-(J4-Pin_6)
Routing:
- net Net-(J2-Pin_13): track 101.9 -> 19.4 mm
- net CANL: track 27.0 -> 107.4 mm
- net CANH: track 22.3 -> 99.5 mm
- net Net-(J2-Pin_14): track 93.6 -> 18.9 mm
- net Net-(J2-Pin_16): track 88.6 -> 16.2 mm
- net Net-(J2-Pin_15): track 85.4 -> 18.1 mm
- net Net-(J2-Pin_17): track 79.1 -> 15.5 mm
- net Net-(J4-Pin_10): track 0.00 -> 54.3 mm
- net Net-(J2-Pin_12): track 72.9 -> 26.8 mm
- net Net-(J4-Pin_6): track 0.00 -> 42.0 mm
- net Net-(J2-Pin_11): track 80.7 -> 43.9 mm
- net Net-(J4-Pin_13): track 33.4 -> 0.00 mm
- net Net-(J4-Pin_14): track 21.8 -> 0.00 mm
- net Net-(J1-Pin_10): track 20.5 -> 4.15 mm
- net GND: track 15.3 -> 5.90 mm, vias 69 -> 164
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