File: FVCU.kicad_sch (KiCad schematic)
At the start: 12 parts, among them J1 ESP32 Connector, J2 Conn_01x19, J3 MCP2551, J4 Conn_01x14

Commit message: Updated
Parts:
- added C1: C, Capacitor_SMD:C_0805_2012Metric_Pad1.18x1.45mm_HandSolder, symbol Device:C
- added R5: 3K, Resistor_SMD:R_0805_2012Metric, symbol Device:R
- added TP1, TP2, TP3, TP4, TP5: TestPoint, TestPoint:TestPoint_Pad_D2.0mm, symbol Connector:TestPoint
Connections:
- net +5V: now also J4.9 (Pin_9), C1.1; no longer J4.1 (Pin_1)
- net CANH: now also J4.11 (Pin_11), TP2.1; no longer J4.3 (Pin_3)
- net CANL: now also J4.12 (Pin_12), TP1.1; no longer J4.4 (Pin_4)
- net GND: now also J1.19 (Pin_19), J4.14 (Pin_14), C1.2, R5.2, TP3.1; no longer J3.8 (Pin_8), J4.2 (Pin_2)
- net at R1.2, R3.1: now also J2.11 (Pin_11), TP4.1; no longer J2.12 (Pin_12)
- net at R3.2: now also J4.10 (Pin_10); no longer J4.14 (Pin_14)
- net at R2.2, R4.1: now also J2.12 (Pin_12), TP5.1; no longer J2.11 (Pin_11)
- net at J2.13 (Pin_13): now also J4.5 (Pin_5); no longer J4.12 (Pin_12)
- net at J2.14 (Pin_14): now also J4.4 (Pin_4); no longer J4.11 (Pin_11)
- net at J2.15 (Pin_15): now also J4.3 (Pin_3); no longer J4.10 (Pin_10)
- net at J2.16 (Pin_16): now also J4.2 (Pin_2); no longer J4.7 (Pin_7)
- net at J2.17 (Pin_17): now also J4.1 (Pin_1); no longer J4.6 (Pin_6)
- net at J4.13 (Pin_13): no longer R4.2
- new net: J3.8 (Pin_8), R5.1
- new net: J4.6 (Pin_6), R4.2
Other:
- moved on the sheet: J4
